File: pcb/dht22.sch (EAGLE design)
At the start: 4 parts, among them IC2 MEGA328P

Commit message: add web
Parts:
- added R2: 4k7, rcl:R-EU_0207/10
- added S1: (no value), switch-omron:10-XX
Connections:
- new net N$1: IC2.PC6(/RESET), R2.1, S1.S1
- net GND: now also S1.P1
- net VCC: now also R2.2
Changed lines of the file:
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@@
 <part name="GND3" library="supply1" deviceset="GND" device=""/>
 <part name="SUPPLY4" library="supply2" deviceset="VCC" device=""/>
+<part name="S1" library="switch-omron" deviceset="10-XX" device=""/>
+<part name="R2" library="rcl" deviceset="R-EU_" device="0207/10" value="4k7"/>
+<part name="SUPPLY6" library="supply2" deviceset="VCC" device=""/>
+<part name="GND4" library="supply1" deviceset="GND" device=""/>
 </parts>
 <sheets>
@@
 <instance part="GND3" gate="1" x="83.82" y="53.34"/>
 <instance part="SUPPLY4" gate="G$1" x="91.44" y="53.34" rot="R90"/>
+<instance part="S1" gate="1" x="17.78" y="88.9" rot="R270"/>
+<instance part="R2" gate="G$1" x="25.4" y="91.44" rot="R90"/>
+<instance part="SUPPLY6" gate="G$1" x="25.4" y="99.06"/>
+<instance part="GND4" gate="1" x="10.16" y="83.82"/>
 </instances>
 <busses>
@@
 <wire x1="93.98" y1="53.34" x2="101.6" y2="53.34" width="0.1524" layer="91"/>
 </segment>
+<segment>
+<pinref part="R2" gate="G$1" pin="2"/>
+<pinref part="SUPPLY6" gate="G$1" pin="VCC"/>
+</segment>
 </net>
 <net name="GND" class="0">
@@
 <pinref part="GND3" gate="1" pin="GND"/>
 <wire x1="83.82" y1="55.88" x2="101.6" y2="55.88" width="0.1524" layer="91"/>
+</segment>
+<segment>
+<pinref part="S1" gate="1" pin="P1"/>
+<pinref part="GND4" gate="1" pin="GND"/>
+<wire x1="10.16" y1="86.36" x2="12.7" y2="86.36" width="0.1524" layer="91"/>
 </segment>
 </net>
@@
 </segment>
 </net>
+<net name="N$1" class="0">
+<segment>
+<pinref part="IC2" gate="G$1" pin="PC6(/RESET)"/>
+<pinref part="S1" gate="1" pin="S1"/>
+<wire x1="22.86" y1="86.36" x2="25.4" y2="86.36" width="0.1524" layer="91"/>
+<pinref part="R2" gate="G$1" pin="1"/>
+<wire x1="25.4" y1="86.36" x2="27.94" y2="86.36" width="0.1524" layer="91"/>
+<junction x="25.4" y="86.36"/>
+</segment>
+</net>
